Commit message: Way too many changes for 1 commit, but I am able to get mass_sim multi_agent.launch to run with the configuration it is at currently. Will wait to rebase the package with RC1.0 branch since it is still being modified.

File: fcu_sim_plugins/xacro/gimbal.xacro (robot description, xacro)
@@ -7,6 +7,8 @@
               parent_link
               camera_topic
+              frame_rate
               pose_topic
               command_topic
+              use_slipring
               *origin">
     <xacro:gimbal_plugin_macro
@@ -14,7 +16,8 @@
       parent_link="${parent_link}"
       camera_topic="${camera_topic}"
+      frame_rate="${frame_rate}"
       pose_topic="${pose_topic}"
       command_topic="${command_topic}"
-      mass="0.001"
+      mass="0.00001"
       x_rotation_range="1000000000"
       y_rotation_range="1000000000"
@@ -28,5 +31,5 @@
   <xacro:macro
     name="gimbal_plugin_macro"
-    params="namespace parent_link camera_topic pose_topic command_topic
+    params="namespace parent_link camera_topic frame_rate pose_topic command_topic
       mass x_rotation_range y_rotation_range z_rotation_range time_constant
       *inertia *origin">
@@ -50,5 +53,5 @@
       <inertial>
         <inertia ixx="0.00001" ixy="0.0" ixz="0.0" iyy="0.00001" iyz="0.0" izz="0.00001" />
-        <mass value="0.0001" />
+        <mass value="${mass}" />
         <origin xyz="0 0 0" rpy = "0 0 0"/>
       </inertial>
@@ -65,5 +68,5 @@
       <inertial>
         <inertia ixx="0.00001" ixy="0.0" ixz="0.0" iyy="0.00001" iyz="0.0" izz="0.00001" />
-        <mass value="0.0001" />
+        <mass value="${mass}" />
         <origin xyz="0 0 0" rpy = "0 0 0"/>
       </inertial>
@@ -80,5 +83,5 @@
       <inertial>
         <inertia ixx="0.00001" ixy="0.0" ixz="0.0" iyy="0.00001" iyz="0.0" izz="0.00001" />
-        <mass value="0.0001" />
+        <mass value="${mass}" />
         <origin xyz="0 0 0" rpy = "0 0 0"/>
       </inertial>
@@ -95,5 +98,5 @@
       <sensor type="camera" name="gimbal/camera">
         <always_on>true</always_on>
-        <update_rate>30</update_rate>
+  <update_rate>${frame_rate}</update_rate>
         <camera>
           <horizontal_fov>2</horizontal_fov>
@@ -108,8 +111,8 @@
           </clip>
         </camera>
-        <plugin name="${namespace}/gimbal_camera" filename="libgazebo_ros_camera.so">
+  <plugin filename="libfcu_sim_camera_plugin.so" name="${namespace}/gimbal_camera">
           <robotNamespace>${namespace}</robotNamespace>
           <alwaysOn>true</alwaysOn>
-          <updateRate>30</updateRate>
+    <updateRate>${frame_rate}</updateRate>
           <cameraName>gimbal/camera</cameraName>
           <imageTopicName>${camera_topic}</imageTopicName>
@@ -134,4 +137,5 @@
         <commandTopic>${command_topic}</commandTopic>
         <poseTopic>${pose_topic}</poseTopic>
+        <useSlipring>${use_slipring}</useSlipring>
       </plugin>
     </gazebo>
